Commit message: Updated my robot

File: src/my_robot_description/urdf/common_properties.xacro (robot description, xacro)
@@ -6,4 +6,7 @@
     <material name="gray">
         <color rgba="0.7 0.7 0.7 1" />
+    </material>
+    <material name="red">
+        <color rgba="1 0 0 1" />
     </material>
     <xacro:macro name="box_inertia" params="m x y z o_xyz o_rpy">

File: src/my_robot_description/urdf/mobile_base.xacro (robot description, xacro)
@@ -79,6 +79,6 @@
     <link name="base_footprint" />
     <joint name="base_joint" type="fixed">
-        <parent link="base_link" />
-        <child link="base_footprint" />
+        <parent link="base_footprint" />
+        <child link="base_link" />
         <origin xyz="0 0 ${wheel_radius}" rpy="0 0 0" />
     </joint>

File: src/my_robot_description/urdf/mobile_base_gazebo.xacro (robot description, xacro)
@@ -1,3 +1,3 @@
-<?xacro version="1.0"?>
+<?xml version="1.0"?>
 <robot xmlns:xacro="http://www.ros.org/wiki/xacro">
     <gazebo reference="caster_wheel_link">
@@ -9,4 +9,7 @@
             <left_joint>base_left_wheel_joint</left_joint>
             <right_joint>base_right_wheel_joint</right_joint>
+            <ros>
+                <remapping>odom:=odom</remapping>
+            </ros>
             <frame_id>odom</frame_id>
             <child_frame_id>base_footprint</child_frame_id>

File: src/my_robot_description/urdf/my_robot.urdf.xacro (robot description, xacro)
@@ -4,3 +4,4 @@
     <xacro:include filename="$(find my_robot_description)/urdf/mobile_base.xacro" />
     <xacro:include filename="$(find my_robot_description)/urdf/mobile_base_gazebo.xacro" />
+    <xacro:include filename="$(find my_robot_description)/urdf/lidar.xacro" />
 </robot>
